File: matrix.sch (KiCad schematic (older format))
At the start: 122 parts

Commit message: More routing
Parts:
- removed D?: D, symbol D
- removed SW?: KEY_MENU, symbol SW_DPST_x2
- added D53, D62, D63, D64: D, cherrymx:DIODE, symbol D
- added SW53: KEY_UP, cherrymx:CHERRY_PCB_100H, symbol SW_DPST_x2
- added SW62: KEY_LEFT, cherrymx:CHERRY_PCB_100H, symbol SW_DPST_x2
- added SW63: KEY_DOWN, cherrymx:CHERRY_PCB_100H, symbol SW_DPST_x2
- added SW64: KEY_RIGHT, cherrymx:CHERRY_PCB_100H, symbol SW_DPST_x2
- D1, D10, D11, D12, D13, D14, D15, D16, D17, D18, D19, D2, D20, D21, D22, D23, D24, D25, D26, D27, D28, D29, D3, D30, D31, D32, D33, D34, D35, D36, D37, D38, D39, D4, D40, D41, D42, D43, D44, D45, D46, D47, D48, D49, D5, D50, D51, D52, D54, D55, D56, D57, D58, D59, D6, D60, D61, D7, D8, D9: renamed from D?; footprint (none) -> cherrymx:DIODE
- SW1, SW10, SW11, SW12, SW13, SW16, SW17, SW18, SW19, SW2, SW20, SW21, SW22, SW23, SW24, SW25, SW26, SW27, SW3, SW30, SW31, SW32, SW33, SW34, SW35, SW36, SW37, SW38, SW39, SW4, SW40, SW43, SW44, SW45, SW46, SW47, SW48, SW49, SW5, SW50, SW51, SW52, SW59, SW6, SW60, SW61, SW7, SW8, SW9: renamed from SW?; footprint (none) -> cherrymx:CHERRY_PCB_100H
- SW14: renamed from SW?; value KEY_EQUAL -> KEY_DELETE; footprint (none) -> cherrymx:CHERRY_PCB_200H
- SW15, SW28: renamed from SW?; footprint (none) -> cherrymx:CHERRY_PCB_150H
- SW29, SW54: renamed from SW?; footprint (none) -> cherrymx:CHERRY_PCB_175H
- SW41, SW42: renamed from SW?; footprint (none) -> cherrymx:CHERRY_PCB_225H
- SW55, SW56, SW57: renamed from SW?; footprint (none) -> cherrymx:CHERRY_PCB_125H
- SW58: renamed from SW?; footprint (none) -> cherrymx:CHERRY_PCB_625H
Connections:
- net col11: now also D62.1 (K)
- net col12: now also D53.1 (K), D63.1 (K); no longer D54.1 (K)
- net col13: now also D54.1 (K), D64.1 (K)
- net row4: now also SW52.1 (A), SW53.1 (A)
- net row5: now also SW62.1 (A), SW63.1 (A), SW64.1 (A)
- new net: D53.2 (A), SW53.2 (B)
- new net: D63.2 (A), SW63.2 (B)
- new net: D62.2 (A), SW62.2 (B)
- new net: D64.2 (A), SW64.2 (B)
Other:
- moved on the sheet: D54, SW54A

Commit message: checkpoint
Connections:
- net col10: now also D60.1 (K)
- net col11: now also D61.1 (K); no longer D62.1 (K)
- net col12: now also D62.1 (K); no longer D63.1 (K)
- net col13: now also D63.1 (K); no longer D64.1 (K)
- net col14: now also D64.1 (K)
- net col4: no longer D58.1 (K)
- net col5: no longer D59.1 (K)
- net col6: now also D58.1 (K); no longer D60.1 (K)
- net col8: no longer D61.1 (K)
- net col9: now also D59.1 (K)
Other:
- moved on the sheet: D58, D59, D60, D61, D62, D63, D64, SW58A, SW59A, SW60A, SW61A, SW62A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
Changed lines of the file:
@@
 L SW_DPST_x2 SW58
 U 1 1 5921C154
-P 3200 5150
-F 0 "SW58" H 3200 5275 50  0000 C CNN
-F 1 "KEY_SPACE" H 3200 5050 50  0000 C CNN
-F 2 "cherrymx:CHERRY_PCB_625H" H 3200 5150 50  0001 C CNN
-F 3 "" H 3200 5150 50  0001 C CNN
-	1    3200 5150
+P 4200 5150
+F 0 "SW58" H 4200 5275 50  0000 C CNN
+F 1 "KEY_SPACE" H 4200 5050 50  0000 C CNN
+F 2 "cherrymx:CHERRY_PCB_625H" H 4200 5150 50  0001 C CNN
+F 3 "" H 4200 5150 50  0001 C CNN
+	1    4200 5150
 	0    1    1    0
 $EndComp
@@
 L D D58
 U 1 1 5921C15A
-P 3350 5450
-F 0 "D58" H 3350 5550 50  0000 C CNN
-F 1 "D" H 3350 5350 50  0000 C CNN
-F 2 "cherrymx:DIODE" H 3350 5450 50  0001 C CNN
-F 3 "" H 3350 5450 50  0001 C CNN
-	1    3350 5450
-	-1   0    0    1
-$EndComp
-$Comp
-L SW_DPST_x2 SW59
-U 1 1 5921C645
-P 3700 5150
-F 0 "SW59" H 3700 5275 50  0000 C CNN
-F 1 "KEY_RALT" H 3700 5050 50  0000 C CNN
-F 2 "cherrymx:CHERRY_PCB_100H" H 3700 5150 50  0001 C CNN
-F 3 "" H 3700 5150 50  0001 C CNN
-	1    3700 5150
-	0    1    1    0
-$EndComp
-$Comp
-L D D59
-U 1 1 5921C64B
-P 3850 5450
-F 0 "D59" H 3850 5550 50  0000 C CNN
-F 1 "D" H 3850 5350 50  0000 C CNN
-F 2 "cherrymx:DIODE" H 3850 5450 50  0001 C CNN
-F 3 "" H 3850 5450 50  0001 C CNN
-	1    3850 5450
-	-1   0    0    1
-$EndComp
-$Comp
-L SW_DPST_x2 SW60
-U 1 1 5921CD21
-P 4200 5150
-F 0 "SW60" H 4200 5275 50  0000 C CNN
-F 1 "KEY_FN" H 4200 5050 50  0000 C CNN
-F 2 "cherrymx:CHERRY_PCB_100H" H 4200 5150 50  0001 C CNN
-F 3 "" H 4200 5150 50  0001 C CNN
-	1    4200 5150
-	0    1    1    0
-$EndComp
-$Comp
-L D D60
-U 1 1 5921CD27
 P 4350 5450
-F 0 "D60" H 4350 5550 50  0000 C CNN
+F 0 "D58" H 4350 5550 50  0000 C CNN
 F 1 "D" H 4350 5350 50  0000 C CNN
 F 2 "cherrymx:DIODE" H 4350 5450 50  0001 C CNN
@@
 $EndComp
 $Comp
+L SW_DPST_x2 SW59
+U 1 1 5921C645
+P 5700 5150
+F 0 "SW59" H 5700 5275 50  0000 C CNN
+F 1 "KEY_RALT" H 5700 5050 50  0000 C CNN
+F 2 "cherrymx:CHERRY_PCB_100H" H 5700 5150 50  0001 C CNN
+F 3 "" H 5700 5150 50  0001 C CNN
+	1    5700 5150
+	0    1    1    0
+$EndComp
+$Comp
+L D D59
+U 1 1 5921C64B
+P 5850 5450
+F 0 "D59" H 5850 5550 50  0000 C CNN
+F 1 "D" H 5850 5350 50  0000 C CNN
+F 2 "cherrymx:DIODE" H 5850 5450 50  0001 C CNN
+F 3 "" H 5850 5450 50  0001 C CNN
+	1    5850 5450
+	-1   0    0    1
+$EndComp
+$Comp
+L SW_DPST_x2 SW60
+U 1 1 5921CD21
+P 6200 5150
+F 0 "SW60" H 6200 5275 50  0000 C CNN
+F 1 "KEY_FN" H 6200 5050 50  0000 C CNN
+F 2 "cherrymx:CHERRY_PCB_100H" H 6200 5150 50  0001 C CNN
+F 3 "" H 6200 5150 50  0001 C CNN
+	1    6200 5150
+	0    1    1    0
+$EndComp
+$Comp
+L D D60
+U 1 1 5921CD27
+P 6350 5450
+F 0 "D60" H 6350 5550 50  0000 C CNN
+F 1 "D" H 6350 5350 50  0000 C CNN
+F 2 "cherrymx:DIODE" H 6350 5450 50  0001 C CNN
+F 3 "" H 6350 5450 50  0001 C CNN
+	1    6350 5450
+	-1   0    0    1
+$EndComp
+$Comp
 L SW_DPST_x2 SW61
 U 1 1 5921E900
-P 5200 5150
-F 0 "SW61" H 5200 5275 50  0000 C CNN
-F 1 "KEY_RCTRL" H 5200 5050 50  0000 C CNN
-F 2 "cherrymx:CHERRY_PCB_100H" H 5200 5150 50  0001 C CNN
-F 3 "" H 5200 5150 50  0001 C CNN
-	1    5200 5150
+P 6650 5150
+F 0 "SW61" H 6650 5275 50  0000 C CNN
+F 1 "KEY_RCTRL" H 6650 5050 50  0000 C CNN
+F 2 "cherrymx:CHERRY_PCB_100H" H 6650 5150 50  0001 C CNN
+F 3 "" H 6650 5150 50  0001 C CNN
+	1    6650 5150
 	0    1    1    0
 $EndComp
@@
 L D D61
 U 1 1 5921E906
-P 5350 5450
-F 0 "D61" H 5350 5550 50  0000 C CNN
-F 1 "D" H 5350 5350 50  0000 C CNN
-F 2 "cherrymx:DIODE" H 5350 5450 50  0001 C CNN
-F 3 "" H 5350 5450 50  0001 C CNN
-	1    5350 5450
+P 6800 5450
+F 0 "D61" H 6800 5550 50  0000 C CNN
+F 1 "D" H 6800 5350 50  0000 C CNN
+F 2 "cherrymx:DIODE" H 6800 5450 50  0001 C CNN
+F 3 "" H 6800 5450 50  0001 C CNN
+	1    6800 5450
 	-1   0    0    1
 $EndComp
@@
 Connection ~ 7200 4200
 Wire Wire Line
-	1300 4900 8800 4900
+	1300 4900 8850 4900
 Wire Wire Line
 	1700 5350 1700 5450
@@
 	2700 5350 2700 5450
 Wire Wire Line
-	2700 4950 2700 4900
+	2700 4900 2700 4950
 Connection ~ 2700 4900
 Wire Wire Line
-	3200 5350 3200 5450
-Wire Wire Line
-	3200 4950 3200 4900
-Connection ~ 3200 4900
-Wire Wire Line
-	3700 5350 3700 5450
-Wire Wire Line
-	3700 4950 3700 4900
-Connection ~ 3700 4900
-Wire Wire Line
 	4200 5350 4200 5450
 Wire Wire Line
-	4200 4900 4200 4950
-Connection ~ 4200 4900
-Wire Wire Line
-	5200 5350 5200 5450
-Wire Wire Line
-	5200 4950 5200 4900
-Connection ~ 5200 4900
+	5700 5350 5700 5450
+Wire Wire Line
+	6200 5350 6200 5450
+Wire Wire Line
+	6650 5350 6650 5450
 Wire Wire Line
 	2000 2500 2000 5650
@@
 Wire Wire Line
 	3500 2500 3500 5650
-Connection ~ 3500 5450
 Connection ~ 3500 4750
 Connection ~ 3500 3950
@@
 Wire Wire Line
 	4000 2500 4000 5650
-Connection ~ 4000 5450
 Connection ~ 4000 4750
 Connection ~ 4000 3950
@@
 Connection ~ 4500 3950
 Connection ~ 4500 4750
-Connection ~ 4500 5450
 Wire Wire Line
 	5000 2500 5000 5650
-Connection ~ 5000 5450
 Connection ~ 5000 4750
 Connection ~ 5000 3950
@@
 Wire Wire Line
 	5500 2500 5500 5650
-Connection ~ 5500 5450
 Connection ~ 5500 4750
 Connection ~ 5500 3950
@@
 L SW_DPST_x2 SW63
 U 1 1 59248D0F
+P 7700 5150
+F 0 "SW63" H 7700 5275 50  0000 C CNN
+F 1 "KEY_DOWN" H 7700 5050 50  0000 C CNN
+F 2 "cherrymx:CHERRY_PCB_100H" H 7700 5150 50  0001 C CNN
+F 3 "" H 7700 5150 50  0001 C CNN
+	1    7700 5150
+	0    1    1    0
+$EndComp
+$Comp
+L D D63
+U 1 1 59248D15
+P 7850 5450
+F 0 "D63" H 7850 5550 50  0000 C CNN
+F 1 "D" H 7850 5350 50  0000 C CNN
+F 2 "cherrymx:DIODE" H 7850 5450 50  0001 C CNN
+F 3 "" H 7850 5450 50  0001 C CNN
+	1    7850 5450
+	-1   0    0    1
+$EndComp
+Wire Wire Line
+	7700 5350 7700 5450
+Connection ~ 7500 4750
+$Comp
+L SW_DPST_x2 SW62
+U 1 1 592494BF
 P 7200 5150
-F 0 "SW63" H 7200 5275 50  0000 C CNN
-F 1 "KEY_DOWN" H 7200 5050 50  0000 C CNN
+F 0 "SW62" H 7200 5275 50  0000 C CNN
+F 1 "KEY_LEFT" H 7200 5050 50  0000 C CNN
 F 2 "cherrymx:CHERRY_PCB_100H" H 7200 5150 50  0001 C CNN
 F 3 "" H 7200 5150 50  0001 C CNN
@@
 $EndComp
 $Comp
-L D D63
-U 1 1 59248D15
+L D D62
+U 1 1 592494C5
 P 7350 5450
-F 0 "D63" H 7350 5550 50  0000 C CNN
+F 0 "D62" H 7350 5550 50  0000 C CNN
 F 1 "D" H 7350 5350 50  0000 C CNN
 F 2 "cherrymx:DIODE" H 7350 5450 50  0001 C CNN
@@
 Wire Wire Line
 	7200 5350 7200 5450
+$Comp
+L SW_DPST_x2 SW64
+U 1 1 59249A11
+P 8200 5150
+F 0 "SW64" H 8200 5275 50  0000 C CNN
+F 1 "KEY_RIGHT" H 8200 5050 50  0000 C CNN
+F 2 "cherrymx:CHERRY_PCB_100H" H 8200 5150 50  0001 C CNN
+F 3 "" H 8200 5150 50  0001 C CNN
+	1    8200 5150
+	0    1    1    0
+$EndComp
+$Comp
+L D D64
+U 1 1 59249A17
+P 8350 5450
+F 0 "D64" H 8350 5550 50  0000 C CNN
+F 1 "D" H 8350 5350 50  0000 C CNN
+F 2 "cherrymx:DIODE" H 8350 5450 50  0001 C CNN
+F 3 "" H 8350 5450 50  0001 C CNN
+	1    8350 5450
+	-1   0    0    1
+$EndComp
+Wire Wire Line
+	8200 5350 8200 5450
+Connection ~ 8000 4750
+Connection ~ 7000 5450
+Connection ~ 8500 5450
+Wire Wire Line
+	8200 4950 8200 4900
+Connection ~ 8200 4900
+Wire Wire Line
+	7700 4950 7700 4900
+Connection ~ 7700 4900
 Wire Wire Line
 	7200 4950 7200 4900
 Connection ~ 7200 4900
-Connection ~ 7500 4750
 Connection ~ 7500 5450
-$Comp
-L SW_DPST_x2 SW62
-U 1 1 592494BF
-P 6700 5150
-F 0 "SW62" H 6700 5275 50  0000 C CNN
-F 1 "KEY_LEFT" H 6700 5050 50  0000 C CNN
-F 2 "cherrymx:CHERRY_PCB_100H" H 6700 5150 50  0001 C CNN
-F 3 "" H 6700 5150 50  0001 C CNN
-	1    6700 5150
-	0    1    1    0
-$EndComp
-$Comp
-L D D62
-U 1 1 592494C5
-P 6850 5450
-F 0 "D62" H 6850 5550 50  0000 C CNN
-F 1 "D" H 6850 5350 50  0000 C CNN
-F 2 "cherrymx:DIODE" H 6850 5450 50  0001 C CNN
-F 3 "" H 6850 5450 50  0001 C CNN
-	1    6850 5450
-	-1   0    0    1
-$EndComp
-Wire Wire Line
-	6700 5350 6700 5450
-Wire Wire Line
-	6700 4950 6700 4900
-Connection ~ 6700 4900
-$Comp
-L SW_DPST_x2 SW64
-U 1 1 59249A11
-P 7700 5150
-F 0 "SW64" H 7700 5275 50  0000 C CNN
-F 1 "KEY_RIGHT" H 7700 5050 50  0000 C CNN
-F 2 "cherrymx:CHERRY_PCB_100H" H 7700 5150 50  0001 C CNN
-F 3 "" H 7700 5150 50  0001 C CNN
-	1    7700 5150
-	0    1    1    0
-$EndComp
-$Comp
-L D D64
-U 1 1 59249A17
-P 7850 5450
-F 0 "D64" H 7850 5550 50  0000 C CNN
-F 1 "D" H 7850 5350 50  0000 C CNN
-F 2 "cherrymx:DIODE" H 7850 5450 50  0001 C CNN
-F 3 "" H 7850 5450 50  0001 C CNN
-	1    7850 5450
-	-1   0    0    1
-$EndComp
-Wire Wire Line
-	7700 5350 7700 5450
-Wire Wire Line
-	7700 4950 7700 4900
-Connection ~ 7700 4900
 Connection ~ 8000 5450
-Connection ~ 8000 4750
-Connection ~ 7000 5450
+Wire Wire Line
+	6650 4950 6650 4900
+Connection ~ 6650 4900
+Wire Wire Line
+	6950 5450 7000 5450
+Wire Wire Line
+	6200 4950 6200 4900
+Connection ~ 6200 4900
+Connection ~ 6500 5450
+Connection ~ 6000 5450
+Wire Wire Line
+	5700 4950 5700 4900
+Connection ~ 5700 4900
+Wire Wire Line
+	4200 4950 4200 4900
+Connection ~ 4200 4900
+Connection ~ 4500 5450
 $EndSCHEMATC
