File: _autosave-keyboard.kicad_pcb (KiCad board)
At the start: 2 copper layers, 297 x 113 mm, 156 parts, among them J1 CONN_01X05, J2 USB_A, J3 CONN_02X03, SW1 KEY_ESC, SW10 KEY_9, SW11 KEY_0, SW12 KEY_MINUS, SW13 KEY_EQUAL, SW14 KEY_DELETE, SW15 KEY_TAB, SW16 KEY_Q, SW17 KEY_W, SW18 KEY_E, SW19 KEY_R, SW2 KEY_1, SW20 KEY_T, SW21 KEY_Y, SW22 KEY_U, SW23 KEY_I, SW24 KEY_O, SW25 KEY_P, SW26 KEY_LBRACK, SW27 KEY_RBRACK, SW28 KEY_BACKSLH, SW29 KEY_CAPS, SW3 KEY_2, SW30 KEY_A, SW31 KEY_S, SW32 KEY_D, SW33 KEY_F, SW34 KEY_G, SW35 KEY_H, SW36 KEY_J, SW37 KEY_K, SW38 KEY_L, SW39 KEY_SEMI, SW4 KEY_3, SW40 KEY_APOS, SW41 KEY_ENTER, SW42 KEY_LSHIFT, SW43 KEY_Z, SW44 KEY_X, SW45 KEY_C, SW46 KEY_V, SW47 KEY_B, SW48 KEY_N, SW49 KEY_M, SW5 KEY_4, SW50 KEY_COMMA, SW51 KEY_PERIOD, SW52 KEY_SLASH, SW53 KEY_UP, SW54 KEY_RSHIFT, SW55 KEY_LCTRL, SW56 KEY_SPECIAL, SW57 KEY_LALT, SW58 KEY_SPACE, SW59 KEY_RALT, SW6 KEY_5, SW60 KEY_FN, SW61 KEY_RCTRL, SW62 KEY_LEFT, SW63 KEY_DOWN, SW64 KEY_RIGHT, SW7 KEY_6, SW8 KEY_7, SW9 KEY_8, U1 ATMEGA32U4-AU, Y1 16mhz

Commit message: Add board edges
Parts:
- added REF**: MountingHole_2.7mm, Mounting_Holes:MountingHole_2.7mm, F.Cu at (104.0, 252.8)
- added REF**: MountingHole_2.7mm, Mounting_Holes:MountingHole_2.7mm, F.Cu at (48.0, 252.2)
- moved REF** 10.1 mm to (190.0, 148.0)
- moved REF** 2.17 mm to (212.1, 252.0)
Other:
- board text added: "AUGUST"
- board text added: "V1.0"
Changed lines of the file:
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@@
     (area 42.049999 143.924999 339.200001 257.075001)
     (thickness 1.6)
-    (drawings 9)
-    (tracks 986)
+    (drawings 11)
+    (tracks 990)
     (zones 0)
-    (modules 156)
+    (modules 158)
     (nets 103)
   )
@@
     (38 B.Mask user)
     (39 F.Mask user)
-    (40 Dwgs.User user)
+    (40 Dwgs.User user hide)
     (41 Cmts.User user)
     (42 Eco1.User user)
@@
   )
   (module Mounting_Holes:MountingHole_2.7mm (layer F.Cu)
+    (at 103.975 252.794)
+    (descr "Mounting Hole 2.7mm, no annular")
+    (tags "mounting hole 2.7mm no annular")
+    (fp_text reference REF** (at 0 -3.7) (layer F.SilkS) hide
+      (effects (font (size 1 1) (thickness 0.15)))
+    )
+    (fp_text value MountingHole_2.7mm (at 0 3.7) (layer F.Fab)
+      (effects (font (size 1 1) (thickness 0.15)))
+    )
+    (fp_circle (center 0 0) (end 2.7 0) (layer Cmts.User) (width 0.15))
+    (fp_circle (center 0 0) (end 2.95 0) (layer F.CrtYd) (width 0.05))
+    (pad 1 np_thru_hole circle (at 0 0) (size 2.7 2.7) (drill 2.7) (layers *.Cu *.Mask))
+  )
+  (module Mounting_Holes:MountingHole_2.7mm (layer F.Cu)
+    (at 47.968 252.159)
+    (descr "Mounting Hole 2.7mm, no annular")
+    (tags "mounting hole 2.7mm no annular")
+    (fp_text reference REF** (at 0 -3.7) (layer F.SilkS) hide
+      (effects (font (size 1 1) (thickness 0.15)))
+    )
+    (fp_text value MountingHole_2.7mm (at 0 3.7) (layer F.Fab)
+      (effects (font (size 1 1) (thickness 0.15)))
+    )
+    (fp_circle (center 0 0) (end 2.7 0) (layer Cmts.User) (width 0.15))
+    (fp_circle (center 0 0) (end 2.95 0) (layer F.CrtYd) (width 0.05))
+    (pad 1 np_thru_hole circle (at 0 0) (size 2.7 2.7) (drill 2.7) (layers *.Cu *.Mask))
+  )
+  (module Mounting_Holes:MountingHole_2.7mm (layer F.Cu)
     (at 276.06 253.048)
     (descr "Mounting Hole 2.7mm, no annular")
@@
   )
   (module Mounting_Holes:MountingHole_2.7mm (layer F.Cu)
-    (at 200.114 148)
+    (at 190 148)
     (descr "Mounting Hole 2.7mm, no annular")
     (tags "mounting hole 2.7mm no annular")
@@
   )
   (module Mounting_Holes:MountingHole_2.7mm (layer F.Cu)
-    (at 211.29 250)
+    (at 212.052 252.032)
     (descr "Mounting Hole 2.7mm, no annular")
     (tags "mounting hole 2.7mm no annular")
@@
     (pad HOLE np_thru_hole circle (at 5.08 0) (size 1.7018 1.7018) (drill 1.7018) (layers *.Cu))
   )
+  (gr_text V1.0 (at 306.159 252.159) (layer F.SilkS)
+    (effects (font (size 3 3) (thickness 0.3)))
+  )
+  (gr_text AUGUST (at 254.216 252.159) (layer F.SilkS)
+    (effects (font (size 3 3) (thickness 0.3)))
+  )
   (gr_line (start 339.125 148) (end 335.125 144) (angle 90) (layer Edge.Cuts) (width 0.15))
   (gr_line (start 339.125 253) (end 339.125 148) (angle 90) (layer Edge.Cuts) (width 0.15))
@@
     (effects (font (size 1.5 1.5) (thickness 0.3)) (justify mirror))
   )
-  (segment (start 149.06 248.73) (end 153.124 252.794) (width 0.4) (layer F.Cu) (net 1))
-  (segment (start 197.32 252.794) (end 209.766 240.348) (width 0.4) (layer F.Cu) (net 1))
-  (segment (start 153.124 252.794) (end 197.32 252.794) (width 0.4) (layer F.Cu) (net 1))
-  (segment (start 46.19 154.75) (end 48.222 152.718) (width 0.4) (layer B.Cu) (net 1))
-  (segment (start 52.54 251.27) (end 118.58 251.27) (width 0.4) (layer B.Cu) (net 1))
+  (segment (start 46.19 244.92) (end 46.19 245.301) (width 0.4) (layer B.Cu) (net 1))
   (segment (start 46.19 154.75) (end 46.19 197.93) (width 0.4) (layer B.Cu) (net 1))
   (segment (start 46.19 197.93) (end 46.19 244.92) (width 0.4) (layer B.Cu) (net 1))
-  (segment (start 46.19 244.92) (end 52.54 251.27) (width 0.4) (layer B.Cu) (net 1))
-  (segment (start 118.58 251.27) (end 127.978 251.27) (width 0.4) (layer B.Cu) (net 1))
   (segment (start 130.01 251.27) (end 127.978 251.27) (width 0.4) (layer B.Cu) (net 1))
   (segment (start 59.904 152.718) (end 61.682 150.94) (width 0.4) (layer B.Cu) (net 1))
   (segment (start 48.222 152.718) (end 59.904 152.718) (width 0.4) (layer B.Cu) (net 1))
+  (segment (start 46.19 154.75) (end 48.222 152.718) (width 0.4) (layer B.Cu) (net 1))
+  (segment (start 125.311 251.27) (end 127.978 251.27) (width 0.4) (layer B.Cu) (net 1))
+  (segment (start 121.12 247.079) (end 125.311 251.27) (width 0.4) (layer B.Cu) (net 1))
+  (segment (start 47.968 247.079) (end 121.12 247.079) (width 0.4) (layer B.Cu) (net 1))
+  (segment (start 46.19 245.301) (end 47.968 247.079) (width 0.4) (layer B.Cu) (net 1))
+  (segment (start 149.06 248.73) (end 153.124 252.794) (width 0.4) (layer F.Cu) (net 1))
+  (segment (start 197.32 252.794) (end 209.766 240.348) (width 0.4) (layer F.Cu) (net 1))
+  (segment (start 153.124 252.794) (end 197.32 252.794) (width 0.4) (layer F.Cu) (net 1))
   (segment (start 61.682 149.416) (end 63.586 149.416) (width 0.4) (layer B.Cu) (net 1))
   (segment (start 63.586 149.416) (end 64.732 148.27) (width 0.4) (layer B.Cu) (net 1))
@@
   (segment (start 314.16 215.71) (end 318.065 215.71) (width 0.25) (layer B.Cu) (net 82))
   (segment (start 318.065 215.71) (end 319.815 217.46) (width 0.25) (layer B.Cu) (net 82))
-  (segment (start 52.032 252.54) (end 129.756 252.54) (width 0.4) (layer B.Cu) (net 83))
-  (segment (start 44.92 245.428) (end 52.032 252.54) (width 0.4) (layer B.Cu) (net 83))
+  (segment (start 44.92 245.428) (end 47.46 247.968) (width 0.4) (layer B.Cu) (net 83))
   (segment (start 44.92 222.568) (end 44.92 172.276) (width 0.4) (layer B.Cu) (net 83))
   (segment (start 48.476 150.94) (end 44.92 154.496) (width 0.4) (layer B.Cu) (net 83))
@@
   (segment (start 132.296 255.08) (end 141.44 255.08) (width 0.4) (layer B.Cu) (net 83))
   (segment (start 129.756 252.54) (end 132.296 255.08) (width 0.4) (layer B.Cu) (net 83))
+  (segment (start 125.184 252.54) (end 129.756 252.54) (width 0.4) (layer B.Cu) (net 83))
+  (segment (start 120.612 247.968) (end 125.184 252.54) (width 0.4) (layer B.Cu) (net 83))
+  (segment (start 47.46 247.968) (end 120.612 247.968) (width 0.4) (layer B.Cu) (net 83))
   (segment (start 160.49 229.68) (end 198.082 229.68) (width 0.4) (layer F.Cu) (net 83))
   (segment (start 198.082 235.268) (end 209.766 235.268) (width 0.4) (layer F.Cu) (net 83))
