File: keyboard.kicad_pcb (KiCad board)
At the start: 2 copper layers, 297 x 113 mm, 156 parts, among them J1 CONN_01X05, J2 USB_A, J3 CONN_02X03, SW1 KEY_ESC, SW10 KEY_9, SW11 KEY_0, SW12 KEY_MINUS, SW13 KEY_EQUAL, SW14 KEY_DELETE, SW15 KEY_TAB, SW16 KEY_Q, SW17 KEY_W, SW18 KEY_E, SW19 KEY_R, SW2 KEY_1, SW20 KEY_T, SW21 KEY_Y, SW22 KEY_U, SW23 KEY_I, SW24 KEY_O, SW25 KEY_P, SW26 KEY_LBRACK, SW27 KEY_RBRACK, SW28 KEY_BACKSLH, SW29 KEY_CAPS, SW3 KEY_2, SW30 KEY_A, SW31 KEY_S, SW32 KEY_D, SW33 KEY_F, SW34 KEY_G, SW35 KEY_H, SW36 KEY_J, SW37 KEY_K, SW38 KEY_L, SW39 KEY_SEMI, SW4 KEY_3, SW40 KEY_APOS, SW41 KEY_ENTER, SW42 KEY_LSHIFT, SW43 KEY_Z, SW44 KEY_X, SW45 KEY_C, SW46 KEY_V, SW47 KEY_B, SW48 KEY_N, SW49 KEY_M, SW5 KEY_4, SW50 KEY_COMMA, SW51 KEY_PERIOD, SW52 KEY_SLASH, SW53 KEY_UP, SW54 KEY_RSHIFT, SW55 KEY_LCTRL, SW56 KEY_SPECIAL, SW57 KEY_LALT, SW58 KEY_SPACE, SW59 KEY_RALT, SW6 KEY_5, SW60 KEY_FN, SW61 KEY_RCTRL, SW62 KEY_LEFT, SW63 KEY_DOWN, SW64 KEY_RIGHT, SW7 KEY_6, SW8 KEY_7, SW9 KEY_8, U1 ATMEGA32U4-AU, Y1 16mhz

Commit message: fab
Parts:
- added REF**: MountingHole_2.7mm, Mounting_Holes:MountingHole_2.7mm, F.Cu at (104.0, 252.8)
- added REF**: MountingHole_2.7mm, Mounting_Holes:MountingHole_2.7mm, F.Cu at (48.0, 252.2)
- SW42: footprint cherrymx:CHERRY_PLATE_200H -> cherrymx:CHERRY_PCB_200H
- moved REF** 10.1 mm to (190.0, 148.0)
- moved REF** 2.17 mm to (212.1, 252.0)
Connections:
- R1 pad 2: /RES -> /RST
- U1 pad 13: /RES -> /RST
Routing:
- net /RST: track 0.00 -> 82.5 mm, vias 0 -> 1
- net /SCK: track 483.0 -> 472.6 mm, vias 1 -> 0
- net /RES: track 5.66 -> 0.00 mm
- net /matrix/col2: track 141.8 -> 145.0 mm
Other:
- board text added: "AUGUST"
- board text added: "V1.0"
